File: HW2/board.sch (EAGLE design)
At the start: 21 parts, among them J1 USB-MB-H

Commit message: board to check
Parts:
- removed U$5: CLOCKCLOCK, lib1:CLOCKCLOCK
- added CLOCK: CLOCK, lib1:CLOCK
- added J3: (no value), lib1:CONN_08"
- C5, C6: device lib1:CPOL-USB45181B -> lib1:CPOL-USB45181A
- PICKIT3: device lib1:CONN_06NO_SILK_FEMALE_PTH -> lib1:CONN_05
- R3, R4: value 10k -> 330
- renumbered U$3 to PB1, U$6 to PB2
Connections:
- removed net N$12: R3.1, U$1.12.RA4
- removed net N$14: PB2.P$1, R1.1, U$1.11.RB4
- removed net N$15: U$1.25RB14
- removed net N$17: U$1.24.RB13
- removed net N$18: J2.5
- removed net N$2: PICKIT3.5
- removed net N$20: J2.4
- removed net N$21: J2.3
- removed net N$3: PICKIT3.4
- removed net N$5: U$1.7.RB3
- removed net N$8: U$1.26.RB15
- new net A4: J2.3, R3.1, U$1.12.RA4
- new net B13: J3.3, U$1.24.RB13
- new net B14: J3.2, U$1.25RB14
- new net B15: J3.1, U$1.26.RB15
- new net B3: J2.5, U$1.7.RB3
- new net B4: J2.4, PB2.PIN1, R1.1, U$1.11.RB4
- new net B7: J3.6, U$1.16.RB7
- new net B8: J3.5, U$1.17.RB8
- new net B9: J3.4, U$1.18.RB9
- new net D+: J1.D+, U$1.21.D+
- new net D-: J1.D-, U$1.22.D-
- new net PGEC: PICKIT3.5, U$1.5.PGEC1
- new net PGED: PICKIT3.4, U$1.4.PGED1
- net +3V3: now also R4.1
- net +5V: now also J3.7; no longer R4.1
- net B2: now also U$1.6.RB2
- net GND: now also CLOCK.2.GND, J3.8, PB1.PIN2, PB2.PIN2; no longer PB1.P$2, PB2.P$2, U$5.2.GND
- net N$1: now also PB1.PIN1; no longer PB1.P$1
- net N$10: now also CLOCK.1.OSC1; no longer U$5.1.OSC1
- net N$11: now also CLOCK.3.OSC2; no longer U$5.3.OSC2
Other:
- moved on the sheet: C5, J1, LED2, R1
